Commit message: visualized position, ypr and vel with rviz and controller

File: src/config/rov.urdf (robot description, URDF)
Before this commit: robot rov, 2 links, 1 joints
Links:
- added link camera; collision cylinder length=0.1 radius=0.05; visual cylinder length=0.1 radius=0.05
- added link camera_base; collision cylinder length=0.1 radius=0.05; visual cylinder length=0.1 radius=0.05
- added link light_1; collision cylinder length=0.1 radius=0.05; visual cylinder length=0.1 radius=0.05
- added link light_2; collision cylinder length=0.1 radius=0.05; visual cylinder length=0.1 radius=0.05
- added link light_twin; collision box size=0.1 0.05 0.05; visual box size=0.1 0.05 0.05
- added link thruster_1; collision cylinder length=0.1 radius=0.05; visual cylinder length=0.1 radius=0.05
- added link thruster_2; collision cylinder length=0.1 radius=0.05; visual cylinder length=0.1 radius=0.05
- added link thruster_3; collision cylinder length=0.1 radius=0.05; visual cylinder length=0.1 radius=0.05
- added link thruster_4; collision cylinder length=0.1 radius=0.05; visual cylinder length=0.1 radius=0.05
- added link thruster_vertical; collision cylinder length=0.1 radius=0.05; visual cylinder length=0.1 radius=0.05
- link base_link: geometry collision box size=0.5 0.5 0.3; visual box size=0.5 0.5 0.3
- link imu_link: geometry collision box size=0.1 0.1 0.1; visual box size=0.1 0.1 0.1
Joints:
- added joint camera_base_joint: type revolute, parent base_link, child camera_base, origin xyz=0.0 0.3 0, axis 0 0 1, limit lower=-1.57 upper=1.57 effort=1 velocity=1
- added joint camera_joint: type revolute, parent camera_base, child camera, origin xyz=0.0 0.0 0.05, axis 1 0 0, limit lower=-1.57 upper=1.57 effort=1 velocity=1
- added joint light_1_joint: type fixed, parent base_link, child light_1, origin xyz=-0.25 0.25 0.2
- added joint light_2_joint: type fixed, parent base_link, child light_2, origin xyz=0.25 0.25 0.2
- added joint light_twin_joint: type fixed, parent base_link, child light_twin, origin xyz=0.0 0.25 0.2
- added joint thruster_1_joint: type fixed, parent base_link, child thruster_1, origin xyz=-0.3 0.3 0
- added joint thruster_2_joint: type fixed, parent base_link, child thruster_2, origin xyz=0.3 0.3 0
- added joint thruster_3_joint: type fixed, parent base_link, child thruster_3, origin xyz=-0.3 -0.3 0
- added joint thruster_4_joint: type fixed, parent base_link, child thruster_4, origin xyz=0.3 -0.3 0
- added joint thruster_vertical_joint: type fixed, parent base_link, child thruster_vertical, origin xyz=1.0 1.0 1.2
- joint imu_joint: origin xyz=0.0 0.0 0.05 -> xyz=0.0 0.0 0.15
